File: Hardware/Double_Slot/Qwiic Pi SHIM_double_slot.sch (EAGLE design)
At the start: 13 parts, among them J1 Qwiic Right Angle, U2 3.3V/600mA

Commit message: singel and double slot versions done
Parts:
- J9: device Qwiic Pi SHIM:SPARKFUN-CONNECTORS_CONN_03X2PISHIM_LOCK_SLOTS -> Qwiic Pi SHIM:SPARKFUN-CONNECTORS_CONN_03X2PISHIM_LOCK_SLOTS_DOUBLE
Changed lines of the file:
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@@
 <part name="FD3" library="SparkFun-Aesthetics" deviceset="FIDUCIAL" device="UFIDUCIAL" value="FIDUCIALUFIDUCIAL"/>
 <part name="FD4" library="SparkFun-Aesthetics" deviceset="FIDUCIAL" device="UFIDUCIAL" value="FIDUCIALUFIDUCIAL"/>
-<part name="J9" library="Qwiic Pi SHIM" deviceset="SPARKFUN-CONNECTORS_CONN_03X2" device="PISHIM_LOCK_SLOTS"/>
+<part name="J9" library="Qwiic Pi SHIM" deviceset="SPARKFUN-CONNECTORS_CONN_03X2" device="PISHIM_LOCK_SLOTS_DOUBLE"/>
 <part name="SUPPLY6" library="SparkFun-PowerSymbols" deviceset="5V" device=""/>
 <part name="GND1" library="SparkFun" deviceset="GND" device=""/>
