File: Hardware/Production/Qwiic Pi SHIM-Panel.brd (EAGLE design)
At the start: 104.9 x 77.5 mm, 387 parts, among them J1 Qwiic Right Angle, J11 Qwiic Right Angle, J13 Qwiic Right Angle, J15 Qwiic Right Angle, J17 Qwiic Right Angle, J19 Qwiic Right Angle, J2 Qwiic Right Angle, J21 Qwiic Right Angle, J23 Qwiic Right Angle, J25 Qwiic Right Angle, J27 Qwiic Right Angle, J29 Qwiic Right Angle, J31 Qwiic Right Angle, J33 Qwiic Right Angle, J35 Qwiic Right Angle, J37 Qwiic Right Angle, J39 Qwiic Right Angle, J4 Qwiic Right Angle, J41 Qwiic Right Angle, J43 Qwiic Right Angle, J45 Qwiic Right Angle, J47 Qwiic Right Angle, J49 Qwiic Right Angle, J51 Qwiic Right Angle, J53 Qwiic Right Angle, J55 Qwiic Right Angle, J57 Qwiic Right Angle, J59 Qwiic Right Angle, J6 Qwiic Right Angle, J61 Qwiic Right Angle, J63 Qwiic Right Angle, J8 Qwiic Right Angle, U1 3.3V/600mA, U10 3.3V/600mA, U11 3.3V/600mA, U12 3.3V/600mA, U13 3.3V/600mA, U14 3.3V/600mA, U15 3.3V/600mA, U16 3.3V/600mA, U17 3.3V/600mA, U18 3.3V/600mA, U19 3.3V/600mA, U2 3.3V/600mA, U20 3.3V/600mA, U21 3.3V/600mA, U22 3.3V/600mA, U23 3.3V/600mA, U24 3.3V/600mA, U25 3.3V/600mA, U26 3.3V/600mA, U27 3.3V/600mA, U28 3.3V/600mA, U29 3.3V/600mA, U3 3.3V/600mA, U30 3.3V/600mA, U31 3.3V/600mA, U32 3.3V/600mA, U4 3.3V/600mA, U5 3.3V/600mA, U6 3.3V/600mA, U7 3.3V/600mA, U8 3.3V/600mA, U9 3.3V/600mA

Commit message: Reverting to tighter spacing (aka v14 or "4MILS")
-updated single brd files, panel files (and production gerbers)
Parts:
- J10, J12, J14, J16, J18, J20, J22, J24, J26, J28, J3, J30, J32, J34, J36, J38, J40, J42, J44, J46, J48, J5, J50, J52, J54, J56, J58, J60, J62, J64, J7, J9: device Qwiic Pi SHIM:SPARKFUN-CONNECTORS_2X3-NS_PISHIM_LOCKING_SLOTS-2MILS -> Qwiic Pi SHIM:SPARKFUN-CONNECTORS_2X3-NS_PISHIM_LOCKING_SLOTS-4MILS
Other:
- board text added: "v14"
- board text removed: "v12"
